File: key55.kicad_sch (KiCad schematic)
At the start: 111 parts, among them K1 KEYSW, K10 KEYSW, K11 KEYSW, K12 KEYSW, K13 KEYSW, K14 KEYSW, K15 KEYSW, K16 KEYSW, K17 KEYSW, K18 KEYSW, K19 KEYSW, K2 KEYSW, K20 KEYSW, K21 KEYSW, K22 KEYSW, K23 KEYSW, K24 KEYSW, K25 KEYSW, K26 KEYSW, K27 KEYSW, K28 KEYSW, K29 KEYSW, K3 KEYSW, K30 KEYSW, K31 KEYSW, K32 KEYSW, K33 KEYSW, K34 KEYSW, K35 KEYSW, K36 KEYSW, K37 KEYSW, K38 KEYSW, K39 KEYSW, K4 KEYSW, K40 KEYSW, K41 KEYSW, K42 KEYSW, K43 KEYSW, K44 KEYSW, K45 KEYSW, K46 KEYSW, K47 KEYSW, K48 KEYSW, K49 KEYSW, K5 KEYSW, K50 KEYSW, K51 KEYSW, K52 KEYSW, K53 KEYSW, K54 KEYSW, K55 KEYSW, K6 KEYSW, K7 KEYSW, K8 KEYSW, K9 KEYSW, U1 ProMicro

Commit message: Key55 V0.1
pcb done
Parts:
- removed D55: D, TheKeebrary:MD_Diode, symbol keyboard_parts:D
- removed K55: KEYSW, Switch_Keyboard_Hotswap_Kailh:SW_Hotswap_Kailh_MX_1.00u, symbol keyboard_parts:KEYSW
- added D48: D, TheKeebrary:MD_Diode, symbol keyboard_parts:D
- added K48: KEYSW, Switch_Keyboard_Hotswap_Kailh:SW_Hotswap_Kailh_MX_2.25u, symbol keyboard_parts:KEYSW
- K49: renamed from K48; footprint Switch_Keyboard_Hotswap_Kailh:SW_Hotswap_Kailh_MX_2.25u -> Switch_Keyboard_Hotswap_Kailh:SW_Hotswap_Kailh_MX_1.00u
- renumbered D48 to D49, D49 to D50, D50 to D51, D51 to D52, D52 to D53, D53 to D54, D54 to D55, K49 to K50, K50 to K51, K51 to K52, K52 to K53, K53 to K54, K54 to K55
Connections:
- net COL14 is gone; now on net COL13: K15.1
- net COL0: now also U1.1 (TX)
- net COL1: now also U1.2 (RX)
- net COL10: now also U1.20 (F4)
- net COL11: now also U1.19 (F5)
- net COL12: now also U1.18 (F6)
- net COL13: now also U1.17 (F7)
- net COL2: now also U1.5 (SDA)
- net COL3: now also U1.6 (SCL)
- net COL4: now also U1.7 (D4)
- net COL5: now also U1.8 (C6), K48.1
- net COL6: now also U1.9 (D7)
- net COL7: now also U1.10 (E6)
- net COL8: now also U1.11 (B4)
- net COL9: now also U1.12 (B5)
- net ROW0: now also U1.16 (B1); no longer D15.1
- net ROW1: now also U1.15 (B3)
- net ROW2: now also U1.14 (B2)
- net ROW3: now also D15.1, U1.13 (B6), D48.1
- new net: D48.2, K48.2
